Commit message: description pkg >> gazebo classic

File: wbot_description/urdf/wbot.urdf.xacro (robot description, xacro)
@@ -1,10 +1,10 @@
 <?xml version="1.0"?>
-<robot name="bumperbot" xmlns:xacro="http://ros.org/wiki/xacro">
+<robot name="wbot" xmlns:xacro="http://ros.org/wiki/xacro">
   <!-- load proper version of ros2 control -->
-  <xacro:arg name="is_ignition" default="true"/>
+  <xacro:arg name="is_classic" default="true"/>
   <!-- Include Gazebo Parameters -->
-  <xacro:include filename="$(find bumperbot_description)/urdf/bumperbot_gazebo.xacro" />
+  <xacro:include filename="$(find wbot_description)/urdf/wbot_gazebo.xacro" />
   <!-- ros2 control -->
-  <xacro:include filename="$(find bumperbot_description)/urdf/bumperbot_ros2_control.xacro" />
+  <xacro:include filename="$(find wbot_description)/urdf/wbot_ros2_control.xacro" />
   <link name="base_footprint"/>
   <link name="base_link">
@@ -19,5 +19,5 @@
       <origin xyz="0 0 0" rpy="0 0 0" />
       <geometry>
-        <mesh filename="package://bumperbot_description/meshes/base_link.STL" />
+        <mesh filename="package://wbot_description/meshes/base_link.STL" />
       </geometry>
     </visual>
@@ -25,5 +25,5 @@
       <origin xyz="0 0 0" rpy="0 0 0" />
       <geometry>
-        <mesh filename="package://bumperbot_description/meshes/base_link.STL" />
+        <mesh filename="package://wbot_description/meshes/base_link.STL" />
       </geometry>
     </collision>
@@ -45,5 +45,5 @@
       <origin xyz="0 0 0" rpy="1.57 0 0" />
       <geometry>
-        <mesh filename="package://bumperbot_description/meshes/wheel_right_link.STL" />
+        <mesh filename="package://wbot_description/meshes/wheel_right_link.STL" />
       </geometry>
     </visual>
@@ -73,5 +73,5 @@
       <origin xyz="0 0 0" rpy="-1.57 0 0" />
       <geometry>
-        <mesh filename="package://bumperbot_description/meshes/wheel_left_link.STL" />
+        <mesh filename="package://wbot_description/meshes/wheel_left_link.STL" />
       </geometry>
     </visual>
@@ -100,5 +100,5 @@
       <origin xyz="0 0 0" rpy="0 0 0" />
       <geometry>
-        <mesh filename="package://bumperbot_description/meshes/caster_front_link.STL" />
+        <mesh filename="package://wbot_description/meshes/caster_front_link.STL" />
       </geometry>
     </visual>
@@ -127,5 +127,5 @@
       <origin xyz="0 0 0" rpy="0 0 0" />
       <geometry>
-        <mesh filename="package://bumperbot_description/meshes/caster_rear_link.STL" />
+        <mesh filename="package://wbot_description/meshes/caster_rear_link.STL" />
       </geometry>
     </visual>
@@ -154,5 +154,5 @@
       <origin xyz="0.0 0.0 0.0" rpy="0.0 0.0 0.0"/>
         <geometry>
-          <mesh filename="package://bumperbot_description/meshes/imu_link.STL" scale="1.0"/>
+          <mesh filename="package://wbot_description/meshes/imu_link.STL" scale="1.0"/>
         </geometry>
     </visual>
@@ -160,5 +160,5 @@
        <origin xyz="0.0 0.0 0.0" rpy="0.0 0.0 0.0"/>
         <geometry>
-          <mesh filename="package://bumperbot_description/meshes/imu_link.STL" scale="1.0"/>
+          <mesh filename="package://wbot_description/meshes/imu_link.STL" scale="1.0"/>
         </geometry>
     </collision>

File: wbot_description/urdf/wbot_gazebo.xacro (robot description, xacro)
@@ -1,4 +1,4 @@
 <?xml version="1.0"?>
-<robot name="bumperbot" xmlns:xacro="http://ros.org/wiki/xacro">
+<robot name="wbot" xmlns:xacro="http://ros.org/wiki/xacro">
     <gazebo reference = "wheel_right_link">
         <mu1>100000000000000.0</mu1>
@@ -35,21 +35,18 @@
         <maxVel>0.1</maxVel>
     </gazebo>
+ <!-- ros2_control plugin for Gazebo Classic 11 -->
     <gazebo>
-        <!-- is ignition is set to true checks -->
-        <xacro:if value = "$(arg is_ignition)">
-            <plugin filename="ign_ros2_control-system" name = "ign_ros2_control::IgnitionROS2ControlPlugin">
-                <parameters>$(find bumperbot_controller)/config/bumperbot_controllers.yaml</parameters>
-            </plugin>
-            <plugin filename = "ignition-gazebo-imu-system" name = "ignition::gazebo::systems::Imu">
-            </plugin>
-        </xacro:if>
-        <!-- if you use higher then humble like jazzy -->
-        <xacro:unless value = "$(arg is_ignition)">
-            <plugin filename = "gz_ros2_control-system" name = "gz_ros2_control::GazeboSimROS2ControlPlugin">
-                <parameters>$(find bumperbot_controller)/config/bumperbot_controllers.yaml</parameters>
-            </plugin>
-            <plugin filename = "gz-sim-imu-system" name = "gz::sim::systems::Imu">
-            </plugin>
-        </xacro:unless>
+        <plugin name="gazebo_ros2_control" filename="libgazebo_ros2_control.so">
+            <robotNamespace>/</robotNamespace>
+            <robotParam>/robot_description</robotParam>
+            <controlPeriod>0.001</controlPeriod>
+        </plugin>
+        <!-- IMU plugin for Gazebo Classic 11 -->
+        <plugin name="gazebo_ros_imu_sensor" filename="libgazebo_ros_imu_sensor.so">
+            <rosTopic>/imu</rosTopic>
+            <frameName>imu_link</frameName>
+            <updateRate>100.0</updateRate>
+            <gaussianNoise>0.0017</gaussianNoise>
+        </plugin>
     </gazebo>
     <gazebo reference = "imu_link">

File: wbot_description/urdf/wbot_ros2_control.xacro (robot description, xacro)
@@ -1,15 +1,15 @@
 <?xml version="1.0"?>
-<robot name="bumperbot" xmlns:xacro="http://ros.org/wiki/xacro">
-    <ros2_control name = "RobotSystem" type = "system">
-        <xacro:if value = "$(arg is_ignition)">
-        <!-- you are on ros2 humble -->
+<robot name="wbot" xmlns:xacro="http://ros.org/wiki/xacro">
+    <ros2_control name="RobotSystem" type="system">
+        <!-- If using Gazebo Classic 11  -->
+        <xacro:if value="$(arg is_classic)">
             <hardware>
-                <plugin>ign_ros2_control/IgnitionSystem</plugin>
+            <plugin>gazebo_ros2_control/GazeboSimSystem</plugin>
             </hardware>
         </xacro:if>
-    <!-- you are on ros2 jazzy then this will be used -->
-        <xacro:unless value = "$(arg is_ignition)">
+        <!-- Otherwise, using Gazebo Sim / Ignition -->
+        <xacro:unless value="$(arg is_classic)">
             <hardware>
-                <plugin>gz_ros2_control/GazeboSimSystem</plugin>
+            <plugin>gz_ros2_control/GazeboSystem</plugin>
             </hardware>
         </xacro:unless>

Commit message: gazebo wbot launchable

File: wbot_description/urdf/wbot.urdf.xacro (robot description, xacro)
@@ -154,5 +154,5 @@
       <origin xyz="0.0 0.0 0.0" rpy="0.0 0.0 0.0"/>
         <geometry>
-          <mesh filename="package://wbot_description/meshes/imu_link.STL" scale="1.0"/>
+          <mesh filename="package://wbot_description/meshes/imu_link.STL" scale="1.0 1.0 1.0"/>
         </geometry>
     </visual>
@@ -160,5 +160,5 @@
        <origin xyz="0.0 0.0 0.0" rpy="0.0 0.0 0.0"/>
         <geometry>
-          <mesh filename="package://wbot_description/meshes/imu_link.STL" scale="1.0"/>
+          <mesh filename="package://wbot_description/meshes/imu_link.STL" scale="1.0 1.0 1.0"/>
         </geometry>
     </collision>

File: wbot_description/urdf/wbot_gazebo.xacro (robot description, xacro)
@@ -41,11 +41,9 @@
             <robotParam>/robot_description</robotParam>
             <controlPeriod>0.001</controlPeriod>
-        </plugin>
-        <!-- IMU plugin for Gazebo Classic 11 -->
-        <plugin name="gazebo_ros_imu_sensor" filename="libgazebo_ros_imu_sensor.so">
-            <rosTopic>/imu</rosTopic>
-            <frameName>imu_link</frameName>
-            <updateRate>100.0</updateRate>
-            <gaussianNoise>0.0017</gaussianNoise>
+            <ros2_control>
+                <!-- <param name="robot_description" /> -->
+                <!-- <ros2_control_config>$(find wbot_description)/config/ros2_controllers.yaml</ros2_control_config> -->
+                <param name="control_config" value="package://wbot_description/config/ros2_controllers.yaml"/>
+            </ros2_control>
         </plugin>
     </gazebo>
@@ -53,6 +51,6 @@
         <sensor name="imu" type="imu" update_rate="100">
         <always_on>true</always_on>
-        <gz_frame_id>imu_link</gz_frame_id>
-        <topic>imu</topic>
+        <!-- <gz_frame_id>imu_link</gz_frame_id>
+        <topic>imu</topic> -->
         <imu>
             <angular_velocity>
@@ -97,4 +95,10 @@
             </linear_acceleration>
         </imu>
+        <plugin name="gazebo_ros_imu_sensor" filename="libgazebo_ros_imu_sensor.so">
+          <topicName>/imu</topicName>
+          <frameName>imu_link</frameName>
+          <updateRate>100.0</updateRate>
+          <gaussianNoise>0.0017</gaussianNoise>
+        </plugin>
         </sensor>
     </gazebo>
