Commit message: debug

File: wbot_description/urdf/wbot_gazebo.xacro (robot description, xacro)
@@ -45,5 +45,6 @@
     </gazebo>
     <gazebo reference = "imu_link">
-        <sensor name="imu" type="imu" update_rate="100">
+        <sensor name="imu" type="imu" >
+        <!-- <sensor name="imu" type="imu" update_rate="100"> -->
         <always_on>true</always_on>
         <!-- <gz_frame_id>imu_link</gz_frame_id>

File: wbot_description/urdf/wbot_ros2_control.xacro (robot description, xacro)
@@ -5,5 +5,5 @@
         <xacro:if value="$(arg is_classic)">
             <hardware>
-            <plugin>gazebo_ros2_control/GazeboSimSystem</plugin>
+            <plugin>gazebo_ros2_control/GazeboSystem</plugin>
             </hardware>
         </xacro:if>
@@ -11,5 +11,5 @@
         <xacro:unless value="$(arg is_classic)">
             <hardware>
-            <plugin>gz_ros2_control/GazeboSystem</plugin>
+            <plugin>gz_ros2_control/GazeboSimSystem</plugin>
             </hardware>
         </xacro:unless>
@@ -34,4 +34,24 @@
             <state_interface name = "velocity"/>
         </joint>
+        <transmission name="wheel_left_trans">
+        <type>transmission_interface/SimpleTransmission</type>
+        <joint name="wheel_left_joint">
+            <hardwareInterface>hardware_interface/VelocityJointInterface</hardwareInterface>
+        </joint>
+        <actuator name="wheel_left_motor">
+            <hardwareInterface>hardware_interface/VelocityJointInterface</hardwareInterface>
+            <mechanicalReduction>1</mechanicalReduction>
+        </actuator>
+        </transmission>
+        <transmission name="wheel_right_trans">
+        <type>transmission_interface/SimpleTransmission</type>
+        <joint name="wheel_right_joint">
+            <hardwareInterface>hardware_interface/VelocityJointInterface</hardwareInterface>
+        </joint>
+        <actuator name="wheel_right_motor">
+            <hardwareInterface>hardware_interface/VelocityJointInterface</hardwareInterface>
+            <mechanicalReduction>1</mechanicalReduction>
+        </actuator>
+        </transmission>
     </ros2_control>
 </robot>
